File: MD-6.kicad_pcb (KiCad board)
At the start: 2 copper layers, 76.2 x 92.7 mm, 160 parts, among them J1 Conn_02x07_Odd_Even, J10 Conn_01x02_Female, J11 Conn_01x02_Female, J12 Conn_01x02_Female, J13 Conn_01x02_Female, J14 Conn_01x02_Female, J15 Conn_01x02_Female, J16 Conn_01x02_Female, J17 Conn_01x02_Female, J18 Conn_01x02_Female, J19 Conn_01x02_Female, J2 Conn_02x07_Odd_Even, J20 Conn_01x02_Female, J21 Conn_01x04_Female, J22 Conn_01x04_Female, J23 Conn_02x04_Odd_Even, J24 Conn_02x04_Odd_Even, J3 Conn_01x02_Male, J4 Conn_01x02_Female, J5 Conn_01x02_Female, J6 Conn_01x02_Female, J7 Conn_01x02_Female, J8 Conn_01x02_Female, J9 Conn_01x02_Female, SW1 SW_Push, U1 MCP2551-I-SN, U10 BD63130AFM, U11 TLP291, U12 TLP291, U13 BD63130AFM, U14 TLP291, U15 TLP291, U16 BD63130AFM, U17 TLP291, U18 TLP291, U19 BD63130AFM, U2 MCP1792-3302H, U20 TLP291, U21 TLP291, U22 BD63130AFM, U23 TLP291, U24 TLP291, U25 BD63130AFM, U26 TLP291, U27 TLP291, U28 BD63130AFM, U29 TLP291, U3 STM32F303K8Tx, U30 TLP291, U31 BD63130AFM, U4 STM32L010F4P6, U5 TLP291, U6 TLP291, U7 L7805, U8 TLP291, U9 TLP291, Y1 16MHz

Commit message: some
Parts:
- D10, D9, J11, J13, J15, J17, J19, J7, J9, R13, R21, R22, R23, R30, R31, R38, R39, R46, R47, U13, U16, U19, U22, U25, U28, U31: moved to B.Cu
- J14, J8, R16: moved to F.Cu
- moved J18 177.0 mm to (74.3, 129.5), turned to -90 degrees
- moved R61 162.3 mm to (86.4, 158.6)
- moved R63 162.3 mm to (94.4, 150.9)
- moved R64 162.3 mm to (96.1, 147.6)
- moved D15 162.3 mm to (82.3, 158.6)
- moved R62 162.3 mm to (104.4, 138.6)
- moved R46 157.5 mm to (106.7, 105.4), turned to 180 degrees
- moved U28 148.0 mm to (90.2, 109.2)
- moved J16 147.3 mm to (88.3, 129.5), turned to -90 degrees
- moved R47 147.1 mm to (103.5, 105.4), turned to 180 degrees
- moved J6 142.5 mm to (132.1, 73.0)
- moved R45 139.4 mm to (105.4, 118.7)
- moved R48 136.1 mm to (118.7, 108.0), turned to -90 degrees
- moved J4 135.0 mm to (132.1, 59.1)
- moved D13 135.0 mm to (105.4, 116.8)
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
Commit message: v0 done
Parts:
- added C12: C_Polarized, Capacitor_SMD:CP_Elec_10x10, F.Cu at (113.7, 57.8)
- added C13: C_Polarized, Capacitor_SMD:CP_Elec_10x10, F.Cu at (113.7, 71.1)
- added C14: C_Polarized, Capacitor_SMD:CP_Elec_10x10, F.Cu at (113.7, 85.1)
- added C15: C_Polarized, Capacitor_SMD:CP_Elec_10x10, F.Cu at (113.7, 98.4)
- added C16: C_Polarized, Capacitor_SMD:CP_Elec_10x10, F.Cu at (113.7, 111.8)
- added C17: C_Polarized, Capacitor_SMD:CP_Elec_10x10, F.Cu at (104.1, 123.2)
- added C18: C_Polarized, Capacitor_SMD:CP_Elec_10x10, F.Cu at (90.2, 111.1)
- added C19: C_Polarized, Capacitor_SMD:CP_Elec_10x10, F.Cu at (78.7, 111.1)
- added C20: 1uF, Capacitor_SMD:C_0603_1608Metric, F.Cu at (62.9, 122.6)
- C1, C8: value 0.1uF -> 1uF
- C11, C6, C7: value 10uF -> 1uF; footprint Capacitor_SMD:C_0805_2012Metric -> Capacitor_SMD:C_0603_1608Metric
- D11, D12, D13, D14, D15, D16, R29, R37, R45, R53, R54, R55, R61, R62, R63, R69, R70, R71: moved to B.Cu
- Y1: footprint Crystal:Crystal_SMD_3225-4Pin_3.2x2.5mm -> Crystal:Crystal_SMD_HC49-SD
- moved R53 109.7 mm to (97.2, 130.8), turned to 90 degrees
- moved D14 109.0 mm to (97.2, 127.6), turned to -90 degrees
- moved R70 106.3 mm to (80.6, 98.4), turned to 180 degrees
- moved C11 103.0 mm to (67.3, 104.8)
- moved R72 103.0 mm to (80.0, 121.9), turned to 90 degrees
- moved C2 100.0 mm to (64.1, 67.3), turned to 180 degrees
- moved R71 97.6 mm to (77.5, 98.4), turned to 180 degrees
- moved U7 95.8 mm to (69.2, 114.9), turned to -90 degrees
- moved R69 95.4 mm to (71.1, 98.4)
- moved C10 95.2 mm to (69.8, 107.3), turned to 180 degrees
- moved C4 89.8 mm to (83.8, 56.5), turned to 180 degrees
- moved D16 88.3 mm to (74.3, 98.4), turned to 180 degrees
- moved R2 83.6 mm to (75.6, 63.5), turned to 90 degrees
- moved C1 79.8 mm to (66.0, 88.9), turned to -90 degrees
- moved C5 78.0 mm to (77.5, 79.4), turned to -90 degrees
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Connections:
- D5 pad 1: unconnected-(D5-Pad1) -> Net-(D6-Pad3)
- D6 pad 3: unconnected-(D6-Pad3) -> Net-(D6-Pad3)
- Y1 pad 1: /OSC_OUT -> /OSC_IN
- Y1 pad 2: GND -> /OSC_OUT
Routing:
- net +5VP: track 0.00 -> 205.9 mm, vias 0 -> 12
- net +5V: track 0.00 -> 127.5 mm, vias 0 -> 5
- net +3V3: track 0.00 -> 97.0 mm, vias 0 -> 4
- net /EN2: track 0.00 -> 89.6 mm, vias 0 -> 8
- net /NRST: track 0.00 -> 58.7 mm, vias 0 -> 4
- net /ACTIVE2: track 0.00 -> 58.5 mm, vias 0 -> 3
- net /EN1: track 0.00 -> 52.4 mm, vias 0 -> 6
- net /T15C2_M52: track 0.00 -> 49.7 mm, vias 0 -> 2
- net /T15C1_M51: track 0.00 -> 46.9 mm, vias 0 -> 2
- net /NeoPixel: track 0.00 -> 42.1 mm, vias 0 -> 2
- net /driver6/IN2P: track 0.00 -> 41.9 mm, vias 0 -> 1
- net /driver6/IN1P: track 0.00 -> 39.1 mm, vias 0 -> 1
- net /SPI_sck: track 0.00 -> 35.3 mm, vias 0 -> 2
- net /ACTIVE1: track 0.00 -> 33.9 mm, vias 0 -> 2
- net /SPI_dat: track 0.00 -> 31.6 mm, vias 0 -> 2
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- added copper zone on B.Cu, net /driver1/OUT1
- added copper zone on B.Cu, net /driver1/OUT2
- added copper zone on B.Cu, net /driver2/OUT1
- added copper zone on B.Cu, net /driver2/OUT2
- added copper zone on B.Cu, net /driver3/OUT1
- added copper zone on B.Cu, net /driver3/OUT2
- added copper zone on B.Cu, net /driver4/OUT1
- added copper zone on B.Cu, net /driver4/OUT2
- added copper zone on B.Cu, net /driver5/OUT1
- added copper zone on B.Cu, net /driver5/OUT2
- added copper zone on B.Cu, net /driver6/OUT1
- added copper zone on B.Cu, net /driver6/OUT2
- added copper zone on B.Cu, net /driver7/OUT1
- added copper zone on B.Cu, net /driver7/OUT2
- added copper zone on B.Cu, net /driver8/OUT1
- added copper zone on B.Cu, net /driver8/OUT2
- added copper zone on B.Cu, net GND
- added copper zone on F.Cu, net GND
- added copper zone on B.Cu, net GNDPWR
- added copper zone on F.Cu, net GNDPWR
- added copper zone on B.Cu, net RNF
- added copper zone on F.Cu, net RNF
- added copper zone on B.Cu, net VCC
- added copper zone on F.Cu, net VCC
Other:
- board text added: "3.3V"
- board text added: "CAN bus"
- board text added: "CLK"
- board text added: "DIO"
- board text added: "GND"
- board text added: "MD-6_v0"
- board text added: "R16"
- board text added: "RX"
- board text added: "SWD MCU1"
- board text added: "SWD MCU2"
- board text added: "TX"
- board text added: "isolated 75W motor driver x8 with CAN interface Designed by paripal github.com/paripalpp/MD-6"
- board text added: "↑power input↑ 7.4V to 22.2V"
