File: MD-6.kicad_sch (KiCad schematic)
At the start: 27 parts, among them J1 Conn_02x07_Odd_Even, SW1 SW_Push, U1 MCP2551-I-SN, U2 STM32F303K8Tx, U3 MCP1792-3302H, U6 L7812, Y1 16MHz

Commit message: some
Parts:
- removed C16, C17: 33uF, Capacitor_SMD:CP_Elec_6.3x7.7, symbol Device:C_Polarized
- removed D3: LED, LED_SMD:LED_0603_1608Metric, symbol Device:LED
- removed D6: 1N4148W, Diode_SMD:D_SOD-123, symbol Device:D
- removed U6: L7812, Package_TO_SOT_SMD:TO-252-2, symbol Regulator_Linear:L7812
- added C9: 0.1uF, Capacitor_SMD:C_0603_1608Metric, symbol Device:C
- added D3, D4, D5, D6, D7, D8: WS2812C, LED_additional:LED_2020Metric_WS2812C_2.0x2.0mm_P1.0mm, symbol LED_additional:WS2812C
- added H1, H2, H3, H4: MountingHole, MountingHole:MountingHole_3.2mm_M3_Pad_Via, symbol Mechanical:MountingHole
- added J10, J12, J14, J16, J18, J20, J4, J6, J8: Conn_01x02_Female, Connector_T_connector:T_connecter_female_horizontal, symbol Connector:Conn_01x02_Female
- added J11, J13, J15, J17, J19, J5, J7, J9: Conn_01x02_Female, Connector_JST:JST_XA_S02B-XASK-1_1x02_P2.50mm_Horizontal, symbol Connector:Conn_01x02_Female
- added J2: Conn_02x07_Odd_Even, Connector_PinHeader_1.27mm:PinHeader_2x07_P1.27mm_Vertical_SMD, symbol Connector_Generic:Conn_02x07_Odd_Even
- added J21, J22: Conn_01x04_Female, Connector_JST:JST_XA_S04B-XASK-1_1x04_P2.50mm_Horizontal, symbol Connector:Conn_01x04_Female
- added J23, J24: Conn_02x04_Odd_Even, Connector_PinHeader_2.54mm:PinHeader_2x04_P2.54mm_Vertical, symbol Connector_Generic:Conn_02x04_Odd_Even
- added J3: Conn_01x02_Male, Connector_T_connector:T_connecter_male_horizontal, symbol Connector:Conn_01x02_Male
- added R5, R6: 330, Resistor_SMD:R_0603_1608Metric, symbol Device:R
- added R7, R8: 1k, Resistor_SMD:R_0603_1608Metric, symbol Device:R
- added U4: STM32L010F4P6, Package_SO:TSSOP-20_4.4x6.5mm_P0.65mm, symbol MCU_ST_STM32L0:STM32L011F4Px
- added U5, U6: TLP291, Package_SO:SOIC-4_4.55x2.6mm_P1.27mm, symbol Isolator:TLP291
- added U7: L7805, Package_TO_SOT_SMD:TO-252-2, symbol Regulator_Linear:L7805
- renumbered C20 to C1, C1 to C2, C2 to C3, C3 to C4, C4 to C5, C5 to C6, C9 to C7, C6 to C8, U3 to U2, U2 to U3
Connections:
- net AHIN is gone; now on net NeoPixel: U3.18 (PA8)
- net +3V3: now also C9.1, J2.3 (Pin_3), J23.1 (Pin_1), J23.2 (Pin_2), J24.1 (Pin_1), J24.2 (Pin_2), U4.16 (VDD), U4.5 (VDDA); no longer R4.2
- net +5V: now also D3.4 (VDD), D4.4 (VDD), D5.4 (VDD), D6.4 (VDD), D7.4 (VDD), D8.4 (VDD), J21.1 (Pin_1), J22.1 (Pin_1)
- net CANH: now also J21.2 (Pin_2), J22.2 (Pin_2)
- net CANL: now also J21.3 (Pin_3), J22.3 (Pin_3)
- net GND: now also R4.1, C9.2, D3.2 (VSS), D4.2 (VSS), D5.2 (VSS), D6.2 (VSS), D7.2 (VSS), D8.2 (VSS), J2.11 (Pin_11), J2.5 (Pin_5), J2.7 (Pin_7), J21.4 (Pin_4), J22.4 (Pin_4), J23.7 (Pin_7), J23.8 (Pin_8), J24.7 (Pin_7), J24.8 (Pin_8), U4.15 (VSS), U5.2, U6.2
- net GNDPWR: now also J20.2 (Pin_2), J3.2 (Pin_2), U5.3, U6.3, U7.2 (GND)
- net NRST: now also J2.12 (Pin_12), U4.4 (NRST)
- net NeoPixel: no longer U3.15 (PB1)
- net VCC: now also J20.1 (Pin_1), J3.1 (Pin_1), U7.1 (IN)
- net T3C2_M32: now reaches U3.10 (PA4)
- net T2C4_M22: now reaches U3.20 (PA10)
- net ACTIVE2: now reaches U3.25 (PA15)
- net ACTIVE2: now also R6.1, U4.12 (PA6)
- net SPI_sck: now reaches U3.26 (PB3)
- net SPI_sck: now also U4.11 (PA5)
- net T2C1_M11: now reaches U3.6 (PA0)
- net T2C2_M12: now reaches U3.7 (PA1)
- net T15C1_M51: now reaches U3.8 (PA2)
- net T15C2_M52: now reaches U3.9 (PA3)
- net at D2.1 (DOUT): now also D3.3 (DIN)
- net +12V renamed +5VP
- net +5VP: now also R7.2, R8.2, U7.3 (OUT)
- net ALIN: no longer names the net of U3.13 (PA7)
- net BHIN renamed T2C3_M21
- net BLIN renamed T3C3_M41
- net DISABLE renamed SPI_dat
- net SPI_dat: now also U4.13 (PA7)
- net PWM_IN1 renamed ACTIVE1
- net ACTIVE1: now also R5.1
- net PWM_IN2 renamed T3C1_M31
- net SWCLK renamed MC1_SWCLK
- net MC1_SWCLK: now also J23.5 (Pin_5)
- net SWDIO renamed MC1_SWDIO
- net MC1_SWDIO: now also J23.3 (Pin_3)
- net VCP_RX renamed MC1_VCP_RX
- net MC1_VCP_RX: now also J23.6 (Pin_6)
- net VCP_TX renamed MC1_VCP_TX
- net MC1_VCP_TX: now also J23.4 (Pin_4)
- new net: D3.1 (DOUT), D4.3 (DIN)
- new net: R5.2, U5.1
- new net: R4.2, U4.1 (PB9)
- new net: D6.1 (DOUT), D7.3 (DIN)
- new net: R6.2, U6.1
- new net: D4.1 (DOUT), D5.3 (DIN)
- new net: D7.1 (DOUT), D8.3 (DIN)
- new net EN1: R7.1, U5.4
- new net EN2: R8.1, U6.4
- new net MC2_SWCLK: J2.6 (Pin_6), J24.5 (Pin_5), U4.20 (PA14)
- new net MC2_SWDIO: J2.4 (Pin_4), J24.3 (Pin_3), U4.19 (PA13)
- new net MC2_VCP_RX: J2.13 (Pin_13), J24.6 (Pin_6), U4.9 (PA3)
- new net MC2_VCP_TX: J2.14 (Pin_14), J24.4 (Pin_4), U4.10 (PA4)
- new net T21C1_M81: U4.18 (PA10)
- new net T21C2_M82: U4.17 (PA9)
- new net T2C1_M61: U4.6 (PA0)
- new net T2C2_M62: U4.7 (PA1)
- new net T2C3_M71: U4.8 (PA2)
- new net T2C4_M72: U4.14 (PB1)
- new net T3C4_M42: U3.15 (PB1)
- new net driver1/OUT1: J4.1 (Pin_1), J5.1 (Pin_1)
- new net driver1/OUT2: J4.2 (Pin_2), J5.2 (Pin_2)
- new net driver2/OUT1: J6.1 (Pin_1), J7.1 (Pin_1)
- new net driver2/OUT2: J6.2 (Pin_2), J7.2 (Pin_2)
- new net driver3/OUT1: J8.1 (Pin_1), J9.1 (Pin_1)
- new net driver3/OUT2: J8.2 (Pin_2), J9.2 (Pin_2)
- new net driver4/OUT1: J10.1 (Pin_1), J11.1 (Pin_1)
- new net driver4/OUT2: J10.2 (Pin_2), J11.2 (Pin_2)
- new net driver5/OUT1: J12.1 (Pin_1), J13.1 (Pin_1)
- new net driver5/OUT2: J12.2 (Pin_2), J13.2 (Pin_2)
- new net driver6/OUT1: J14.1 (Pin_1), J15.1 (Pin_1)
- new net driver6/OUT2: J14.2 (Pin_2), J15.2 (Pin_2)
- new net driver7/OUT1: J16.1 (Pin_1), J17.1 (Pin_1)
- new net driver7/OUT2: J16.2 (Pin_2), J17.2 (Pin_2)
- new net driver8/OUT1: J18.1 (Pin_1), J19.1 (Pin_1)
- new net driver8/OUT2: J18.2 (Pin_2), J19.2 (Pin_2)
Other:
- added sheet driver1 (driver1.kicad_sch)
- added sheet driver2 (driver1.kicad_sch)
- added sheet driver3 (driver1.kicad_sch)
- added sheet driver4 (driver1.kicad_sch)
- added sheet driver5 (driver1.kicad_sch)
- added sheet driver6 (driver1.kicad_sch)
- added sheet driver7 (driver1.kicad_sch)
- added sheet driver8 (driver1.kicad_sch)
- moved on the sheet: C1, C10, C11, C6, C7, D1, D2, U2

Commit message: v0 done
Parts:
- removed Y1: 16MHz, Crystal:Crystal_SMD_3225-4Pin_3.2x2.5mm, symbol Device:Crystal_GND24
- added C20: 1uF, Capacitor_SMD:C_0603_1608Metric, symbol Device:C
- added Y1: 16MHz, Crystal:Crystal_SMD_HC49-SD, symbol Device:Crystal
- C1, C8: value 0.1uF -> 1uF
- C11, C6, C7: value 10uF -> 1uF; footprint Capacitor_SMD:C_0805_2012Metric -> Capacitor_SMD:C_0603_1608Metric
Connections:
- net +5V: now also C20.1
- net GND: now also C20.2
- net OSC_IN: now also Y1.1
- net OSC_OUT: now also Y1.2
- net at D6.3 (DIN): now also D5.1 (DOUT)
Other:
- moved on the sheet: D6, D7, D8
