File: driver1.kicad_sch (KiCad schematic)
At the start: 13 parts, among them U10 BD63130AFM, U8 TLP291, U9 TLP291

Commit message: v0 done
Parts:
- C12: footprint (none) -> Capacitor_SMD:CP_Elec_10x10
Changed lines of the file:
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@@
       (effects (font (size 1.27 1.27)) (justify left))
     )
-    (property "Footprint" "" (id 2) (at 126.6952 121.92 0)
+    (property "Footprint" "Capacitor_SMD:CP_Elec_10x10" (id 2) (at 126.6952 121.92 0)
       (effects (font (size 1.27 1.27)) hide)
     )
